File: PCBs/router/router.kicad_pcb (KiCad board)
At the start: 2 copper layers, 95.3 x 110 mm, 37 parts, among them J1 Conn_01x06_Male, J10 Conn_01x06_Male, J11 Conn_01x06_Male, J12 Conn_01x06_Male, J13 Conn_01x06_Male, J14 Conn_01x06_Male, J15 Conn_01x06_Male, J2 Conn_01x06_Male, J3 Conn_01x06_Male, J4 Conn_01x06_Male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

Commit message: complete traces
Parts:
- moved C7 20.1 mm to (147.8, 124.0), turned to 0 degrees
- moved C6 20.1 mm to (147.9, 104.6), turned to 0 degrees
- moved Y2 0.51 mm to (150.9, 114.3), turned to 270 degrees
Routing:
- net Net-(C2-Pad1): track 0.00 -> 192.8 mm
- net GND: track 353.8 -> 545.4 mm
- net +9V: track 307.1 -> 394.6 mm
- net Net-(J11-Pad2): track 0.00 -> 83.0 mm
- net Net-(J5-Pad5): track 0.00 -> 83.0 mm, vias 0 -> 3
- net Net-(J8-Pad2): track 0.00 -> 81.7 mm
- net Net-(J5-Pad2): track 0.00 -> 79.9 mm, vias 0 -> 3
- net Net-(J8-Pad5): track 0.00 -> 74.4 mm
- net Net-(J7-Pad2): track 0.00 -> 65.4 mm
- net Net-(J7-Pad3): track 0.00 -> 61.8 mm
- net Net-(J3-Pad2): track 0.00 -> 58.7 mm, vias 0 -> 3
- net Net-(J11-Pad5): track 0.00 -> 58.5 mm
- net Net-(J13-Pad2): track 0.00 -> 51.3 mm
- net Net-(J3-Pad5): track 0.00 -> 48.0 mm
- net Net-(J13-Pad5): track 0.00 -> 31.6 mm
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